Commit message: simulator model done

File: bosch_arm/bosch_arm_description/bosch_arm.urdf.xacro (robot description, xacro)
@@ -6,7 +6,8 @@
        name="bosch_arm" >
   <include filename="$(find bosch_arm_description)/urdf/base/base.urdf.xacro" />
+<!--
   <include filename="$(find pr2_description)/gazebo/gazebo.urdf.xacro" />
-  <!-- materials for visualization -->
+   materials for visualization -->
   <include filename="$(find pr2_description)/urdf/materials.urdf.xacro" />
-  <xacro:bosch_arm_base name="base"/>
+  <xacro:bosch_arm name="base"/>
 </robot>

File: bosch_arm/bosch_arm_description/urdf/base/base.gazebo.xacro (robot description, xacro)
@@ -4,33 +4,19 @@
        xmlns:interface="http://playerstage.sourceforge.net/gazebo/xmlschema/#interface"
        xmlns:xacro="http://ros.org/wiki/xacro">
-  <xacro:macro name="pr2_wheel_gazebo_v0" params="suffix parent">
-    <gazebo reference="${parent}_${suffix}_wheel_link">
-      <mu1 value="100.0" />
-      <mu2 value="100.0" />
-      <kp  value="1000000.0" />
-      <kd  value="1.0" />
+  <xacro:macro name="bosch_arm_gazebo" params="name">
+    <gazebo reference="${name}_link">
+      <selfCollide>true</selfCollide>
     </gazebo>
-  </xacro:macro>
-  <xacro:macro name="pr2_caster_gazebo_v0" params="suffix">
-    <gazebo reference="${suffix}_caster_rotation_link">
-      <material value="PR2/caster_texture" />
+    <gazebo reference="${name}_link1">
+      <selfCollide>true</selfCollide>
     </gazebo>
-  </xacro:macro>
-  <xacro:macro name="pr2_base_gazebo_v0" params="name">
-    <gazebo reference="${name}_link">
-      <selfCollide>false</selfCollide>
-      <sensor:contact name="${name}_contact_sensor">
-        <geom>${name}_link_geom</geom>
-        <updateRate>100.0</updateRate>
-        <controller:gazebo_ros_bumper name="${name}_gazebo_ros_bumper_controller" plugin="libgazebo_ros_bumper.so">
-          <alwaysOn>true</alwaysOn>
-          <updateRate>100.0</updateRate>
-          <bumperTopicName>${name}_bumper</bumperTopicName>
-          <interface:bumper name="${name}_bumper_iface" />
-        </controller:gazebo_ros_bumper>
-      </sensor:contact>
+    <gazebo reference="${name}_link2">
+      <selfCollide>true</selfCollide>
     </gazebo>
-    <gazebo reference="${name}_bellow_link">
-      <material value="PR2/Black" />
+    <gazebo reference="${name}_link3">
+      <selfCollide>true</selfCollide>
+    </gazebo>
+    <gazebo reference="${name}_link4">
+      <selfCollide>true</selfCollide>
     </gazebo>
     <gazebo>

File: bosch_arm/bosch_arm_description/urdf/base/base.urdf.xacro (robot description, xacro)
@@ -4,6 +4,6 @@
        xmlns:interface="http://playerstage.sourceforge.net/gazebo/xmlschema/#interface"
        xmlns:xacro="http://ros.org/wiki/xacro">
+  <include filename="$(find bosch_arm_description)/urdf/base/base.gazebo.xacro" />
 <!--
-  <include filename="$(find bosch_arm)/urdf/base/base.gazebo.xacro" />
   <include filename="$(find bosch_arm)/urdf/base/base.transmission.xacro" />-->
   <!-- DATA SOURCES -->
@@ -13,9 +13,39 @@
   <property name="M_PI" value="3.1415926535897931" />
   <property name="base_mass" value="1" />
+  <property name="link1_mass" value="0.5" />
+  <property name="link2_mass" value="0.1" />
+  <property name="link3_mass" value="0.05" />
+  <property name="link4_mass" value="0.05" />
+  <property name="base_z" value="0.35" />
+  <property name="link3_z" value="0.55145" />
+  <property name="link3_center_z" value="${link3_z/2}" />
+  <property name="link4_center_z" value="0.005545" />
   <!-- The xacro macro xacro:pr2_base contains: base, casters and wheels -->
-  <xacro:macro name="bosch_arm_base" params="name">
+  <xacro:macro name="bosch_arm" params="name">
     <link name="${name}_link">
       <inertial>
         <mass value="${base_mass}" />
+        <origin xyz="0 0 ${base_z}" />
+        <inertia ixx="5.652232699207" ixy="-0.009719934438" ixz="1.293988226423"
+                 iyy="5.669473158652" iyz="-0.007379583694" izz="3.683196351726" />
+      </inertial>
+      <visual>
+        <origin xyz="0 0 ${base_z}" rpy="${M_PI/2} 0 0" />
+        <geometry>
+          <mesh filename="package://bosch_arm_description/meshes/base-simple.stl" />
+          <!--mesh filename="package://bosch_arm_description/meshes/entire-simple.stl" /-->
+        </geometry>
+        <material name="White" />
+      </visual>
+      <collision>
+        <origin xyz="0 0 ${base_z}" rpy="${M_PI/2} 0 0" />
+        <geometry>
+          <mesh filename="package://bosch_arm_description/meshes/base-simple.stl" />
+        </geometry>
+      </collision>
+    </link>
+    <link name="${name}_link1">
+      <inertial>
+        <mass value="${link1_mass}" />
         <origin xyz="0 0 0" />
         <inertia ixx="5.652232699207" ixy="-0.009719934438" ixz="1.293988226423"
@@ -25,17 +55,119 @@
         <origin xyz="0 0 0" rpy="0 0 0" />
         <geometry>
-          <mesh filename="package://bosch_arm_description/meshes/base.stl" />
-        </geometry>
-        <material name="White" />
-      </visual>
-      <collision>
-        <origin xyz="0 0 0" rpy="0 0 0" />
-        <geometry>
-          <mesh filename="package://bosch_arm_description/meshes/caster_L.stl" />
-        </geometry>
-      </collision>
-    </link>
+          <mesh filename="package://bosch_arm_description/meshes/joint1-simple.stl" />
+          <!--mesh filename="package://bosch_arm_description/meshes/entire-simple.stl" /-->
+        </geometry>
+        <material name="White" />
+      </visual>
+      <collision>
+        <origin xyz="0 0 0" rpy="0 0 0" />
+        <geometry>
+          <mesh filename="package://bosch_arm_description/meshes/joint1-simple.stl" />
+        </geometry>
+      </collision>
+    </link>
+    <link name="${name}_link2">
+      <inertial>
+        <mass value="${link2_mass}" />
+        <origin xyz="0 0 0" />
+        <inertia ixx="5.652232699207" ixy="-0.009719934438" ixz="1.293988226423"
+                 iyy="5.669473158652" iyz="-0.007379583694" izz="3.683196351726" />
+      </inertial>
+      <visual>
+        <origin xyz="0 0 0" rpy="0 0 0" />
+        <geometry>
+          <mesh filename="package://bosch_arm_description/meshes/joint2-simple.stl" />
+          <!--mesh filename="package://bosch_arm_description/meshes/entire-simple.stl" /-->
+        </geometry>
+        <material name="White" />
+      </visual>
+      <collision>
+        <origin xyz="0 0 0" rpy="0 0 0" />
+        <geometry>
+          <mesh filename="package://bosch_arm_description/meshes/joint2-simple.stl" />
+        </geometry>
+      </collision>
+    </link>
+    <link name="${name}_link3">
+      <inertial>
+        <mass value="${link3_mass}" />
+        <origin xyz="0 0 ${link3_center_z}" />
+        <inertia ixx="0.652232699207" ixy="-0.009719934438" ixz="1.293988226423"
+                 iyy="0.669473158652" iyz="-0.007379583694" izz="3.683196351726" />
+      </inertial>
+      <visual>
+        <origin xyz="0 0 0" rpy="0 0 0" />
+        <geometry>
+          <mesh filename="package://bosch_arm_description/meshes/joint3-simple.stl" />
+        </geometry>
+        <material name="White" />
+      </visual>
+      <collision>
+        <origin xyz="0 0 0" rpy="0 0 0" />
+        <geometry>
+          <mesh filename="package://bosch_arm_description/meshes/joint3-simple.stl" />
+        </geometry>
+      </collision>
+    </link>
+    <link name="${name}_link4">
+      <inertial>
+        <mass value="${link4_mass}" />
+        <origin xyz="0 0 ${link4_center_z}" />
+        <inertia ixx="0.652232699207" ixy="-0.009719934438" ixz="1.293988226423"
+                 iyy="0.669473158652" iyz="-0.007379583694" izz="3.683196351726" />
+      </inertial>
+      <visual>
+        <origin xyz="0 0 0" rpy="0 0 0" />
+        <geometry>
+          <mesh filename="package://bosch_arm_description/meshes/joint4-simple.stl" />
+        </geometry>
+        <material name="White" />
+      </visual>
+      <collision>
+        <origin xyz="0 0 0" rpy="0 0 0" />
+        <geometry>
+          <mesh filename="package://bosch_arm_description/meshes/joint4-simple.stl" />
+        </geometry>
+      </collision>
+    </link>
+    <joint name="${name}_joint1" type="revolute">
+      <axis xyz="0 0 1" />
+      <origin xyz="0 0 ${base_z}" rpy="${M_PI/2} 0 0" />
+      <limit effort="100" velocity="100" lower="${-M_PI/2}" upper="${M_PI/2}" /> <!-- alpha tested velocity and effort limits -->
+      <safety_controller  k_velocity="10" />
+      <!--calibration rising="${ref_position}" /-->
+      <dynamics damping="0.0" friction="0.0" />
+      <parent link="${name}_link"/>
+      <child link="${name}_link1" />
+    </joint>
+    <joint name="${name}_joint2" type="revolute">
+      <axis xyz="0 0 1" />
+      <origin xyz="0 0 0" rpy=" 0 ${M_PI/2} 0" />
+      <limit effort="100" velocity="100" lower="${-M_PI/2}" upper="${M_PI/2}"/> <!-- alpha tested velocity and effort limits -->
+      <safety_controller  k_velocity="10" />
+      <dynamics damping="0.0" friction="0.0" />
+      <parent link="${name}_link1"/>
+      <child link="${name}_link2" />
+    </joint>
+    <joint name="${name}_joint3" type="revolute">
+      <axis xyz="0 0 1" />
+      <origin xyz=" 0 0 0" rpy="${-M_PI/2} 0 0" />
+      <limit effort="100" velocity="100" lower="${-M_PI/2}" upper="${M_PI/2}" /> <!-- alpha tested velocity and effort limits -->
+      <safety_controller  k_velocity="10" />
+      <dynamics damping="0.0" friction="0.0" />
+      <parent link="${name}_link2"/>
+      <child link="${name}_link3" />
+    </joint>
+    <joint name="${name}_joint4" type="continuous">
+      <axis xyz="0 0 1" />
+      <origin xyz="0 -0.04405 ${link3_z}" rpy="0 ${M_PI/2} ${M_PI}" />
+      <limit effort="100" velocity="100"/>
+      <safety_controller  k_velocity="10" />
+      <dynamics damping="0.0" friction="0.0" />
+      <parent link="${name}_link3"/>
+      <child link="${name}_link4" />
+    </joint>
     <!-- base_footprint is a fictitious link(frame) that is on the ground right below base_link origin,
-         navigation stack dedpends on this frame -->
+         navigation stack dedpends on this frame >
     <link name="${name}_footprint">
       <inertial>
@@ -52,7 +184,7 @@
         <material name="White" />
       </visual>
-      <collision>
+      <collision-->
         <!-- represent base collision with a simple rectangular model, positioned by base_size_z s.t. top
-             surface of the collision box matches the top surface of the PR2 base -->
+             surface of the collision box matches the top surface of the PR2 base >
         <origin xyz="0 0 0" rpy="0 0 0" />
         <geometry>
@@ -65,35 +197,7 @@
       <child link="${name}_link" />
       <parent link="${name}_footprint"/>
-    </joint>
-    <!-- visualize bellow -->
-    <link name="${name}_bellow_link">
-      <inertial>
-        <mass value="1.0" />
-        <origin xyz="0 0 0" />
-        <inertia ixx="0.01" ixy="0.0" ixz="0.0"
-                 iyy="0.01" iyz="0.0" izz="0.01" />
-      </inertial>
-      <visual>
-        <origin xyz="0 0 0" rpy="0 0 0" />
-        <geometry>
-          <box size="0.05 0.37 0.3" />
-        </geometry>
-        <material name="Black" />
-      </visual>
-      <collision>
-        <origin xyz="0 0 0" rpy="0 0 0" />
-        <geometry>
-          <box size="0.05 0.37 0.3" />
-        </geometry>
-        <material name="Black" />
-      </collision>
-    </link>
-    <joint name="${name}_bellow_joint" type="fixed">
-      <origin xyz="-0.29 0 0.8" rpy="0 0 0" />
-      <parent link="${name}_link" />
-      <child link="${name}_bellow_link"/>
-    </joint>
+    </joint-->
     <!-- gazebo extensions -->
-    <xacro:bosch_arm_base_gazebo name="${name}" />
+    <xacro:bosch_arm_gazebo name="${name}" />
   </xacro:macro>
 </robot>
