Commit message: a

File: bosch_arm/bosch_arm_description/bosch_arm.urdf.xacro (robot description, xacro)
@@ -6,8 +6,5 @@
        name="bosch_arm" >
   <include filename="$(find bosch_arm_description)/urdf/base/base.urdf.xacro" />
-<!--
-  <include filename="$(find pr2_description)/gazebo/gazebo.urdf.xacro" />
-   materials for visualization -->
-  <include filename="$(find pr2_description)/urdf/materials.urdf.xacro" />
-  <xacro:bosch_arm name="base"/>
+  <include filename="$(find bosch_arm_description)/urdf/materials.urdf.xacro" />
+  <xacro:bosch_arm name="bosch_arm"/>
 </robot>

File: bosch_arm/bosch_arm_description/urdf/base/base.gazebo.xacro (robot description, xacro)
@@ -28,5 +28,5 @@
         <gaussianNoise>0.01</gaussianNoise>
         <frameName>map</frameName>
-        <xyzOffsets>25.7 25.7 0</xyzOffsets> <!-- initialize odometry for fake localization-->
+        <xyzOffsets>0 1.23 0</xyzOffsets> <!-- initialize odometry for fake localization-->
         <rpyOffsets>0 0 0</rpyOffsets>
         <interface:position name="p3d_base_position"/>

File: bosch_arm/bosch_arm_description/urdf/base/base.transmission.xacro (robot description, xacro)
@@ -4,20 +4,10 @@
        xmlns:interface="http://playerstage.sourceforge.net/gazebo/xmlschema/#interface"
        xmlns:xacro="http://ros.org/wiki/xacro">
-  <!--  Caster wheel transmission
-  <xacro:macro name="pr2_wheel_transmission_v0" params="suffix parent reflect">
-    <transmission type="pr2_mechanism_model/SimpleTransmission" name="${parent}_${suffix}_wheel_trans">
-      <actuator name="${parent}_${suffix}_wheel_motor" />
-      <joint name="${parent}_${suffix}_wheel_joint" />
-      <mechanicalReduction>${reflect * 624/35 * 80/18}</mechanicalReduction>
+  <xacro:macro name="bosch_arm_joint_transmission" params="name suffix">
+    <transmission type="pr2_mechanism_model/SimpleTransmission" name="${name}_joint${suffix}_trans">
+      <actuator name="${name}_joint${suffix}_motor" />
+      <joint name="${name}_joint${suffix}" />
+      <mechanicalReduction>1</mechanicalReduction>
     </transmission>
   </xacro:macro>
-  <!-- Hub transmission only
-  <xacro:macro name="pr2_caster_transmission_v0" params="suffix">
-    <transmission type="pr2_mechanism_model/SimpleTransmission" name="${suffix}_rotation_trans">
-      <actuator name="${suffix}_rotation_motor" />
-      <joint name="${suffix}_rotation_joint" />
-      <mechanicalReduction>${-1 * 624/35 * 80/18}</mechanicalReduction>
-    </transmission>
-  </xacro:macro>
--->
 </robot>

File: bosch_arm/bosch_arm_description/urdf/base/base.urdf.xacro (robot description, xacro)
@@ -5,172 +5,36 @@
        xmlns:xacro="http://ros.org/wiki/xacro">
   <include filename="$(find bosch_arm_description)/urdf/base/base.gazebo.xacro" />
-<!--
-  <include filename="$(find bosch_arm)/urdf/base/base.transmission.xacro" />-->
+  <include filename="$(find bosch_arm_description)/urdf/base/base.transmission.xacro" />
   <!-- DATA SOURCES -->
-  <!-- all link offsets, CG, limits are obtained from Function Engineering spreadsheet 090224_link_data.xls unless stated otherwise -->
   <!-- all link geometry sizes are obtained from Function provided CAD model unless stated otherwise -->
   <!-- all simplified collision geometry are hand approximated from CAD model, sometimes from respective bounding boxes -->
   <property name="M_PI" value="3.1415926535897931" />
-  <property name="base_mass" value="1" />
-  <property name="link1_mass" value="0.5" />
-  <property name="link2_mass" value="0.1" />
-  <property name="link3_mass" value="0.05" />
-  <property name="link4_mass" value="0.05" />
+  <property name="base_mass" value="5.743031" />
+  <property name="base_cm_x" value="-0.000694" />
+  <property name="base_cm_y" value="-0.218533" />
+  <property name="base_cm_z" value="-0.000038" />
+  <property name="link1_mass" value="0.744800" />
+  <property name="link1_cm_x" value="0" />
+  <property name="link1_cm_y" value="0" />
+  <property name="link1_cm_z" value="0" />
+  <property name="link2_mass" value="0.104379" />
+  <property name="link2_cm_x" value="0" />
+  <property name="link2_cm_y" value="0.014484" />
+  <property name="link2_cm_z" value="0" />
+  <property name="link3_mass" value="0.091407" />
+  <property name="link3_cm_x" value="0" />
+  <property name="link3_cm_y" value="-0.003365" />
+  <property name="link3_cm_z" value="0.293324" />
+  <property name="link4_mass" value="0.129569" />
+  <property name="link4_cm_x" value="0.006155" />
+  <property name="link4_cm_y" value="0.156038" />
+  <property name="link4_cm_z" value="0" />
   <property name="base_z" value="0.35" />
-  <property name="link3_z" value="0.55145" />
-  <property name="link3_center_z" value="${link3_z/2}" />
-  <property name="link4_center_z" value="0.005545" />
-  <!-- The xacro macro xacro:pr2_base contains: base, casters and wheels -->
+  <property name="link4_y" value="-0.04405" />
+  <property name="link4_z" value="0.55145" />
   <xacro:macro name="bosch_arm" params="name">
-    <link name="${name}_link">
-      <inertial>
-        <mass value="${base_mass}" />
-        <origin xyz="0 0 ${base_z}" />
-        <inertia ixx="5.652232699207" ixy="-0.009719934438" ixz="1.293988226423"
-                 iyy="5.669473158652" iyz="-0.007379583694" izz="3.683196351726" />
-      </inertial>
-      <visual>
-        <origin xyz="0 0 ${base_z}" rpy="${M_PI/2} 0 0" />
-        <geometry>
-          <mesh filename="package://bosch_arm_description/meshes/base-simple.stl" />
-          <!--mesh filename="package://bosch_arm_description/meshes/entire-simple.stl" /-->
-        </geometry>
-        <material name="White" />
-      </visual>
-      <collision>
-        <origin xyz="0 0 ${base_z}" rpy="${M_PI/2} 0 0" />
-        <geometry>
-          <mesh filename="package://bosch_arm_description/meshes/base-simple.stl" />
-        </geometry>
-      </collision>
-    </link>
-    <link name="${name}_link1">
-      <inertial>
-        <mass value="${link1_mass}" />
-        <origin xyz="0 0 0" />
-        <inertia ixx="5.652232699207" ixy="-0.009719934438" ixz="1.293988226423"
-                 iyy="5.669473158652" iyz="-0.007379583694" izz="3.683196351726" />
-      </inertial>
-      <visual>
-        <origin xyz="0 0 0" rpy="0 0 0" />
-        <geometry>
-          <mesh filename="package://bosch_arm_description/meshes/joint1-simple.stl" />
-          <!--mesh filename="package://bosch_arm_description/meshes/entire-simple.stl" /-->
-        </geometry>
-        <material name="White" />
-      </visual>
-      <collision>
-        <origin xyz="0 0 0" rpy="0 0 0" />
-        <geometry>
-          <mesh filename="package://bosch_arm_description/meshes/joint1-simple.stl" />
-        </geometry>
-      </collision>
-    </link>
-    <link name="${name}_link2">
-      <inertial>
-        <mass value="${link2_mass}" />
-        <origin xyz="0 0 0" />
-        <inertia ixx="5.652232699207" ixy="-0.009719934438" ixz="1.293988226423"
-                 iyy="5.669473158652" iyz="-0.007379583694" izz="3.683196351726" />
-      </inertial>
-      <visual>
-        <origin xyz="0 0 0" rpy="0 0 0" />
-        <geometry>
-          <mesh filename="package://bosch_arm_description/meshes/joint2-simple.stl" />
-          <!--mesh filename="package://bosch_arm_description/meshes/entire-simple.stl" /-->
-        </geometry>
-        <material name="White" />
-      </visual>
-      <collision>
-        <origin xyz="0 0 0" rpy="0 0 0" />
-        <geometry>
-          <mesh filename="package://bosch_arm_description/meshes/joint2-simple.stl" />
-        </geometry>
-      </collision>
-    </link>
-    <link name="${name}_link3">
-      <inertial>
-        <mass value="${link3_mass}" />
-        <origin xyz="0 0 ${link3_center_z}" />
-        <inertia ixx="0.652232699207" ixy="-0.009719934438" ixz="1.293988226423"
-                 iyy="0.669473158652" iyz="-0.007379583694" izz="3.683196351726" />
-      </inertial>
-      <visual>
-        <origin xyz="0 0 0" rpy="0 0 0" />
-        <geometry>
-          <mesh filename="package://bosch_arm_description/meshes/joint3-simple.stl" />
-        </geometry>
-        <material name="White" />
-      </visual>
-      <collision>
-        <origin xyz="0 0 0" rpy="0 0 0" />
-        <geometry>
-          <mesh filename="package://bosch_arm_description/meshes/joint3-simple.stl" />
-        </geometry>
-      </collision>
-    </link>
-    <link name="${name}_link4">
-      <inertial>
-        <mass value="${link4_mass}" />
-        <origin xyz="0 0 ${link4_center_z}" />
-        <inertia ixx="0.652232699207" ixy="-0.009719934438" ixz="1.293988226423"
-                 iyy="0.669473158652" iyz="-0.007379583694" izz="3.683196351726" />
-      </inertial>
-      <visual>
-        <origin xyz="0 0 0" rpy="0 0 0" />
-        <geometry>
-          <mesh filename="package://bosch_arm_description/meshes/joint4-simple.stl" />
-        </geometry>
-        <material name="White" />
-      </visual>
-      <collision>
-        <origin xyz="0 0 0" rpy="0 0 0" />
-        <geometry>
-          <mesh filename="package://bosch_arm_description/meshes/joint4-simple.stl" />
-        </geometry>
-      </collision>
-    </link>
-    <joint name="${name}_joint1" type="revolute">
-      <axis xyz="0 0 1" />
-      <origin xyz="0 0 ${base_z}" rpy="${M_PI/2} 0 0" />
-      <limit effort="100" velocity="100" lower="${-M_PI/2}" upper="${M_PI/2}" /> <!-- alpha tested velocity and effort limits -->
-      <safety_controller  k_velocity="10" />
-      <!--calibration rising="${ref_position}" /-->
-      <dynamics damping="0.0" friction="0.0" />
-      <parent link="${name}_link"/>
-      <child link="${name}_link1" />
-    </joint>
-    <joint name="${name}_joint2" type="revolute">
-      <axis xyz="0 0 1" />
-      <origin xyz="0 0 0" rpy=" 0 ${M_PI/2} 0" />
-      <limit effort="100" velocity="100" lower="${-M_PI/2}" upper="${M_PI/2}"/> <!-- alpha tested velocity and effort limits -->
-      <safety_controller  k_velocity="10" />
-      <dynamics damping="0.0" friction="0.0" />
-      <parent link="${name}_link1"/>
-      <child link="${name}_link2" />
-    </joint>
-    <joint name="${name}_joint3" type="revolute">
-      <axis xyz="0 0 1" />
-      <origin xyz=" 0 0 0" rpy="${-M_PI/2} 0 0" />
-      <limit effort="100" velocity="100" lower="${-M_PI/2}" upper="${M_PI/2}" /> <!-- alpha tested velocity and effort limits -->
-      <safety_controller  k_velocity="10" />
-      <dynamics damping="0.0" friction="0.0" />
-      <parent link="${name}_link2"/>
-      <child link="${name}_link3" />
-    </joint>
-    <joint name="${name}_joint4" type="continuous">
-      <axis xyz="0 0 1" />
-      <origin xyz="0 -0.04405 ${link3_z}" rpy="0 ${M_PI/2} ${M_PI}" />
-      <limit effort="100" velocity="100"/>
-      <safety_controller  k_velocity="10" />
-      <dynamics damping="0.0" friction="0.0" />
-      <parent link="${name}_link3"/>
-      <child link="${name}_link4" />
-    </joint>
-    <!-- base_footprint is a fictitious link(frame) that is on the ground right below base_link origin,
-         navigation stack dedpends on this frame >
     <link name="${name}_footprint">
       <inertial>
-        <mass value="1.0" />
+        <mass value="0.01" />
         <origin xyz="0 0 0" />
         <inertia ixx="0.01" ixy="0.0" ixz="0.0"
@@ -182,10 +46,8 @@
           <box size="0.01 0.01 0.01" />
         </geometry>
-        <material name="White" />
-      </visual>
-      <collision-->
-        <!-- represent base collision with a simple rectangular model, positioned by base_size_z s.t. top
-             surface of the collision box matches the top surface of the PR2 base >
-        <origin xyz="0 0 0" rpy="0 0 0" />
+        <material name="Black" />
+      </visual>
+      <collision>
+        <origin xyz="0 0 ${base_z}" rpy="0 0 0" />
         <geometry>
           <box size="0.001 0.001 0.001" />
@@ -193,11 +55,157 @@
       </collision>
     </link>
+    <link name="${name}_link">
+      <inertial>
+        <mass value="${base_mass}" />
+        <origin xyz="${base_cm_x} ${base_cm_y} ${base_cm_z}" />
+        <inertia ixx="0.148153" ixy="-0.000987" ixz="0.000001"
+                 iyy="0.161046" iyz="-0.000028" izz="0.043711" />
+      </inertial>
+      <visual>
+        <origin xyz="0 0 0" rpy="0 0 0" />
+        <geometry>
+          <mesh filename="package://bosch_arm_description/meshes/base-simple.stl" />
+        </geometry>
+        <material name="White" />
+      </visual>
+      <collision>
+        <origin xyz="0 0 0" rpy="0 0 0" />
+        <geometry>
+          <mesh filename="package://bosch_arm_description/meshes/base-simple.stl" />
+        </geometry>
+      </collision>
+    </link>
+    <link name="${name}_link1">
+      <inertial>
+        <mass value="${link1_mass}" />
+        <origin xyz="${link1_cm_x} ${link1_cm_y} ${link1_cm_z}" />
+        <inertia ixx="0.007733" ixy="0" ixz="0"
+                 iyy="0.010218" iyz="0" izz="0.002684" />
+      </inertial>
+      <visual>
+        <origin xyz="0 0 0" rpy="0 0 0" />
+        <geometry>
+          <mesh filename="package://bosch_arm_description/meshes/joint1-simple.stl" />
+        </geometry>
+        <material name="White" />
+      </visual>
+      <collision>
+        <origin xyz="0 0 0" rpy="0 0 0" />
+        <geometry>
+          <mesh filename="package://bosch_arm_description/meshes/joint1-simple.stl" />
+        </geometry>
+      </collision>
+    </link>
+    <link name="${name}_link2">
+      <inertial>
+        <mass value="${link2_mass}" />
+        <origin xyz="${link2_cm_x} ${link2_cm_y} ${link2_cm_z}" />
+        <inertia ixx="0.000205" ixy="0" ixz="0"
+                 iyy="0.000191" iyz="0" izz="0.000048" />
+      </inertial>
+      <visual>
+        <origin xyz="0 0 0" rpy="0 0 0" />
+        <geometry>
+          <mesh filename="package://bosch_arm_description/meshes/joint2-simple.stl" />
+        </geometry>
+        <material name="White" />
+      </visual>
+      <collision>
+        <origin xyz="0 0 0" rpy="0 0 0" />
+        <geometry>
+          <mesh filename="package://bosch_arm_description/meshes/joint2-simple.stl" />
+        </geometry>
+      </collision>
+    </link>
+    <link name="${name}_link3">
+      <inertial>
+        <mass value="${link3_mass}" />
+        <origin xyz="${link3_cm_x} ${link3_cm_y} ${link3_cm_z}" />
+        <inertia ixx="0.002540" ixy="0" ixz="0"
+                 iyy="0.002530" iyz="-0.000077" izz="0.000018" />
+      </inertial>
+      <visual>
+        <origin xyz="0 0 0" rpy="0 0 0" />
+        <geometry>
+          <mesh filename="package://bosch_arm_description/meshes/joint3-simple.stl" />
+        </geometry>
+        <material name="White" />
+      </visual>
+      <collision>
+        <origin xyz="0 0 0" rpy="0 0 0" />
+        <geometry>
+          <mesh filename="package://bosch_arm_description/meshes/joint3-simple.stl" />
+        </geometry>
+      </collision>
+    </link>
+    <link name="${name}_link4">
+      <inertial>
+        <mass value="${link4_mass}" />
+        <origin xyz="${link4_cm_x} ${link4_cm_y} ${link4_cm_z}" />
+        <inertia ixx="0.003878" ixy="0" ixz="0"
+                 iyy="0.000045" iyz="0" izz="0.003917" />
+      </inertial>
+      <visual>
+        <origin xyz="0 0 0" rpy="0 0 0" />
+        <geometry>
+          <mesh filename="package://bosch_arm_description/meshes/joint4-simple.stl" />
+        </geometry>
+        <material name="White" />
+      </visual>
+      <collision>
+        <origin xyz="0 0 0" rpy="0 0 0" />
+        <geometry>
+          <mesh filename="package://bosch_arm_description/meshes/joint4-simple.stl" />
+        </geometry>
+      </collision>
+    </link>
     <joint name="${name}_footprint_joint" type="fixed">
-      <origin xyz="0 0 0" rpy="0 0 0" />
+      <origin xyz="0 0 ${base_z}" rpy="${M_PI/2} 0 0" />
       <child link="${name}_link" />
       <parent link="${name}_footprint"/>
-    </joint-->
+    </joint>
+    <joint name="${name}_joint1" type="revolute">
+      <axis xyz="0 0 1" />
+      <origin xyz="0 0 0" rpy="0 0 0" />
+      <limit effort="100" velocity="100" lower="${-M_PI/2}" upper="${M_PI/2}" /> <!-- alpha tested velocity and effort limits -->
+      <safety_controller  k_velocity="10" />
+      <!--calibration rising="${ref_position}" /-->
+      <dynamics damping="0.0" friction="0.0" />
+      <parent link="${name}_link"/>
+      <child link="${name}_link1" />
+    </joint>
+    <joint name="${name}_joint2" type="revolute">
+      <axis xyz="0 0 1" />
+      <origin xyz="0 0 0" rpy=" 0 ${M_PI/2} 0" />
+      <limit effort="100" velocity="100" lower="${-M_PI/2}" upper="${M_PI/2}"/> <!-- alpha tested velocity and effort limits -->
+      <safety_controller  k_velocity="10" />
+      <dynamics damping="0.0" friction="0.0" />
+      <parent link="${name}_link1"/>
+      <child link="${name}_link2" />
+    </joint>
+    <joint name="${name}_joint3" type="revolute">
+      <axis xyz="0 0 1" />
+      <origin xyz=" 0 0 0" rpy="${-M_PI/2} 0 0" />
+      <limit effort="100" velocity="100" lower="${-M_PI/2}" upper="${M_PI/2}" /> <!-- alpha tested velocity and effort limits -->
+      <safety_controller  k_velocity="10" />
+      <dynamics damping="0.0" friction="0.0" />
+      <parent link="${name}_link2"/>
+      <child link="${name}_link3" />
+    </joint>
+    <joint name="${name}_joint4" type="continuous">
+      <axis xyz="0 0 1" />
+      <origin xyz="0 ${link4_y} ${link4_z}" rpy="0 ${M_PI/2} ${M_PI}" />
+      <limit effort="100" velocity="100"/>
+      <safety_controller  k_velocity="10" />
+      <dynamics damping="0.0" friction="0.0" />
+      <parent link="${name}_link3"/>
+      <child link="${name}_link4" />
+    </joint>
     <!-- gazebo extensions -->
     <xacro:bosch_arm_gazebo name="${name}" />
+    <xacro:bosch_arm_joint_transmission name="${name}" suffix="1"/>
+    <xacro:bosch_arm_joint_transmission name="${name}" suffix="2"/>
+    <xacro:bosch_arm_joint_transmission name="${name}" suffix="3"/>
+    <xacro:bosch_arm_joint_transmission name="${name}" suffix="4"/>
   </xacro:macro>
 </robot>
