Commit message: a

File: bosch_arm/bosch_arm_description/urdf/base/base.urdf.xacro (robot description, xacro)
@@ -33,8 +33,10 @@
   <property name="link4_y" value="-0.04405" />
   <property name="link4_z" value="0.55145" />
+  <property name="link5_x" value="0.01109" />
+  <property name="link5_y" value="0.51477" />
   <xacro:macro name="bosch_arm" params="name">
     <link name="${name}_footprint">
       <inertial>
-        <mass value="0.01" />
+        <mass value="0.001" />
         <origin xyz="0 0 0" />
         <inertia ixx="0.01" ixy="0.0" ixz="0.0"
@@ -160,4 +162,46 @@
       </collision>
     </link>
+    <link name="${name}_link5">
+      <inertial>
+        <mass value="0.001" />
+        <origin xyz="0 0 0" />
+        <inertia ixx="0.003878" ixy="0" ixz="0"
+                 iyy="0.000045" iyz="0" izz="0.003917" />
+      </inertial>
+      <visual>
+        <origin xyz="0 0 0" rpy="0 0 0" />
+        <geometry>
+          <box size="0.001 0.001 0.001" />
+        </geometry>
+        <material name="White" />
+      </visual>
+      <collision>
+        <origin xyz="0 0 0" rpy="0 0 0" />
+        <geometry>
+          <box size="0.001 0.001 0.001" />
+        </geometry>
+      </collision>
+    </link>
+    <link name="${name}_link6">
+      <inertial>
+        <mass value="0.001" />
+        <origin xyz="0 0 0" />
+        <inertia ixx="0.003878" ixy="0" ixz="0"
+                 iyy="0.000045" iyz="0" izz="0.003917" />
+      </inertial>
+      <visual>
+        <origin xyz="0 0 0" rpy="0 0 0" />
+        <geometry>
+          <box size="0.001 0.001 0.001" />
+        </geometry>
+        <material name="White" />
+      </visual>
+      <collision>
+        <origin xyz="0 0 0" rpy="0 0 0" />
+        <geometry>
+          <box size="0.001 0.001 0.001" />
+        </geometry>
+      </collision>
+    </link>
     <joint name="${name}_footprint_joint" type="fixed">
       <origin xyz="0 0 ${base_z}" rpy="${M_PI/2} 0 0" />
@@ -201,4 +245,22 @@
       <parent link="${name}_link3"/>
       <child link="${name}_link4" />
+    </joint>
+    <joint name="${name}_joint5" type="fixed">
+      <axis xyz="0 0 1" />
+      <origin xyz="${link5_x} ${link5_y} 0" rpy="0 0 0" />
+      <limit effort="100" velocity="100"/>
+      <safety_controller  k_velocity="10" />
+      <dynamics damping="0.0" friction="0.0" />
+      <parent link="${name}_link4"/>
+      <child link="${name}_link5" />
+    </joint>
+    <joint name="${name}_joint6" type="fixed">
+      <axis xyz="0 0 1" />
+      <origin xyz="0 0 0" rpy="0 0 0" />
+      <limit effort="100" velocity="100"/>
+      <safety_controller  k_velocity="10" />
+      <dynamics damping="0.0" friction="0.0" />
+      <parent link="${name}_link5"/>
+      <child link="${name}_link6" />
     </joint>
     <!-- gazebo extensions -->

Commit message: add actuator urdf

File: bosch_arm/bosch_arm_description/urdf/base/base.urdf.xacro (robot description, xacro)
@@ -6,4 +6,5 @@
   <include filename="$(find bosch_arm_description)/urdf/base/base.gazebo.xacro" />
   <include filename="$(find bosch_arm_description)/urdf/base/base.transmission.xacro" />
+  <include filename="$(find bosch_arm_description)/urdf/base/actuator.info.xacro" />
   <!-- DATA SOURCES -->
   <!-- all link geometry sizes are obtained from Function provided CAD model unless stated otherwise -->
@@ -35,4 +36,8 @@
   <property name="link5_x" value="0.01109" />
   <property name="link5_y" value="0.51477" />
+      <property name="r1" value="0.062811565304088" />
+    <property name="r2" value="0.12524850894632" />
+    <property name="r3" value="15.9206349206349" />
+    <property name="r4" value="7.98412698412698" />
   <xacro:macro name="bosch_arm" params="name">
     <link name="${name}_footprint">
@@ -246,5 +251,5 @@
       <child link="${name}_link4" />
     </joint>
-    <joint name="${name}_joint5" type="fixed">
+    <!--joint name="${name}_joint5" type="fixed">
       <axis xyz="0 0 1" />
       <origin xyz="${link5_x} ${link5_y} 0" rpy="0 0 0" />
@@ -254,6 +259,6 @@
       <parent link="${name}_link4"/>
       <child link="${name}_link5" />
-    </joint>
-    <joint name="${name}_joint6" type="fixed">
+    </joint-->
+    <!--joint name="${name}_joint6" type="fixed">
       <axis xyz="0 0 1" />
       <origin xyz="0 0 0" rpy="0 0 0" />
@@ -263,5 +268,5 @@
       <parent link="${name}_link5"/>
       <child link="${name}_link6" />
-    </joint>
+    </joint-->
     <!-- gazebo extensions -->
     <xacro:bosch_arm_gazebo name="${name}" />
@@ -270,4 +275,20 @@
     <xacro:bosch_arm_joint_transmission name="${name}" suffix="3"/>
     <xacro:bosch_arm_joint_transmission name="${name}" suffix="4"/>
+    <xacro:actuator_macro name="actuator1" cmd_addr="1" encoder_addr="1"/>
+    <xacro:actuator_macro name="actuator2" cmd_addr="2" encoder_addr="2"/>
+    <xacro:actuator_macro name="actuator3" cmd_addr="3" encoder_addr="3"/>
+    <xacro:actuator_macro name="actuator4" cmd_addr="4" encoder_addr="4"/>
+    <joint_to_motor_transmission>
+      ${r3}, 0.0, 0.0, 0.0,
+       ${r4},  ${r4}, 0.0, 0.0,
+       ${r4},  ${r4},  ${r4}, 0.0,
+      0.0, 0.0, 0.0,  ${r4}
+    </joint_to_motor_transmission>
+    <motor_to_joint_transmission>
+      ${r1}, 0.0, 0.0, 0.0,
+      -${r1},  ${r2}, 0.0, 0.0,
+      0.0, -${r2},  ${r2}, 0.0,
+      0.0, 0.0, 0.0,  ${r2}
+    </motor_to_joint_transmission>
   </xacro:macro>
 </robot>
