Commit message: add wrapper

File: bosch_arm/bosch_arm_description/urdf/base/base.transmission.xacro (robot description, xacro)
@@ -6,5 +6,5 @@
   <xacro:macro name="bosch_arm_joint_transmission" params="name suffix">
     <transmission type="pr2_mechanism_model/SimpleTransmission" name="${name}_joint${suffix}_trans">
-      <actuator name="${name}_joint${suffix}_motor" />
+      <actuator name="${name}${suffix}" />
       <joint name="${name}_joint${suffix}" />
       <mechanicalReduction>1</mechanicalReduction>

File: bosch_arm/bosch_arm_description/urdf/base/base.urdf.xacro (robot description, xacro)
@@ -167,5 +167,5 @@
       </collision>
     </link>
-    <link name="${name}_link5">
+    <!--link name="${name}_link5">
       <inertial>
         <mass value="0.001" />
@@ -187,6 +187,6 @@
         </geometry>
       </collision>
-    </link>
-    <link name="${name}_link6">
+    </link-->
+    <!--link name="${name}_link6">
       <inertial>
         <mass value="0.001" />
@@ -208,5 +208,5 @@
         </geometry>
       </collision>
-    </link>
+    </link-->
     <joint name="${name}_footprint_joint" type="fixed">
       <origin xyz="0 0 ${base_z}" rpy="${M_PI/2} 0 0" />
@@ -271,8 +271,10 @@
     <!-- gazebo extensions -->
     <xacro:bosch_arm_gazebo name="${name}" />
+    <!--
     <xacro:bosch_arm_joint_transmission name="${name}" suffix="1"/>
     <xacro:bosch_arm_joint_transmission name="${name}" suffix="2"/>
     <xacro:bosch_arm_joint_transmission name="${name}" suffix="3"/>
     <xacro:bosch_arm_joint_transmission name="${name}" suffix="4"/>
+    -->
     <xacro:actuator_macro name="actuator1" cmd_addr="1" encoder_addr="1"/>
     <xacro:actuator_macro name="actuator2" cmd_addr="2" encoder_addr="2"/>
